Commit message: fix pm01

File: source/whole_body_tracking/whole_body_tracking/assets/hightorque/pm01/urdf/pm01_24dof.urdf (robot description, URDF)
Before this commit: robot pm01_24dof, 25 links, 24 joints
Links:
- added link link_elbow_end_l, mass 0.001; collision sphere radius=0.02
- added link link_elbow_end_r, mass 0.001; collision sphere radius=0.02
Joints:
- added joint j17_end_elbow_end_l_joint: type fixed, parent link_elbow_yaw_l, child link_elbow_end_l, origin xyz=0 0 0 rpy=0 0 0
- added joint j22_end_elbow_end_r_joint: type fixed, parent link_elbow_yaw_r, child link_elbow_end_r, origin xyz=0 0 0 rpy=0 0 0
- joint j12_waist_yaw_joint: limit lower=-1.57 upper=1.57 effort=61 velocity=10.0 -> lower=-4.014 upper=1.57 effort=61 velocity=10.0; origin xyz=0 0 0.1 rpy=0 0 0 -> xyz=0.01216 0 0.0809 rpy=0 0 0
- joint j13_shoulder_pitch_l_joint: axis 0 1 0 -> 0 0.998027 0.0627908; limit lower=-1.57 upper=1.57 effort=61 velocity=10.0 -> lower=-2.9671 upper=2.7925 effort=61 velocity=10.0; origin xyz=0.1 0.15 0.1 rpy=0 0 0 -> xyz=-0.027105 0.12916 0.21549 rpy=0 0 0
- joint j14_shoulder_roll_l_joint: limit lower=-1.57 upper=1.57 effort=61 velocity=10.0 -> lower=-0.6108 upper=2.3562 effort=61 velocity=10.0; origin xyz=0 0 0 rpy=0 0 0 -> xyz=-0.0371 0.066941 -0.020838 rpy=0 0 0
- joint j15_shoulder_yaw_l_joint: axis 0 0 1 -> 0 -0.0628027 0.998026; limit lower=-1.57 upper=1.57 effort=61 velocity=10.0 -> lower=-2.618 upper=2.618 effort=61 velocity=10.0; origin xyz=0 0 0 rpy=0 0 0 -> xyz=0.0371 0.017645 -0.070132 rpy=0 0 0
- joint j16_elbow_pitch_l_joint: axis 0 1 0 -> 0.00272431 0.998022 0.0628031; limit lower=-1.57 upper=1.57 effort=61 velocity=10.0 -> lower=-2.1948 upper=0.7374 effort=61 velocity=10.0; origin xyz=0 0 -0.2 rpy=0 0 0 -> xyz=0 0.0065994 -0.10487 rpy=0 0 0
- joint j17_elbow_yaw_l_joint: axis 0 0 1 -> -0.214789 -0.0619207 0.974696; limit lower=-1.57 upper=1.57 effort=61 velocity=10.0 -> lower=-2.618 upper=2.618 effort=61 velocity=10.0; origin xyz=0 0 0 rpy=0 0 0 -> xyz=0.013817 0.0097723 -0.1547 rpy=0 0 0
- joint j18_shoulder_pitch_r_joint: axis 0 1 0 -> 0 0.998027 -0.0627908; limit lower=-1.57 upper=1.57 effort=61 velocity=10.0 -> lower=-2.9671 upper=2.7925 effort=61 velocity=10.0; origin xyz=0.1 -0.15 0.1 rpy=0 0 0 -> xyz=-0.027105 -0.12916 0.21549 rpy=0 0 0
- joint j19_shoulder_roll_r_joint: limit lower=-1.57 upper=1.57 effort=61 velocity=10.0 -> lower=-2.3562 upper=0.6108 effort=61 velocity=10.0; origin xyz=0 0 0 rpy=0 0 0 -> xyz=-0.0371 -0.066941 -0.020838 rpy=0 0 0
- joint j20_shoulder_yaw_r_joint: axis 0 0 1 -> 0 0.0627908 0.998027; limit lower=-1.57 upper=1.57 effort=61 velocity=10.0 -> lower=-2.618 upper=2.618 effort=61 velocity=10.0; origin xyz=0 0 0 rpy=0 0 0 -> xyz=0.0371 -0.017644 -0.070132 rpy=0 0 0
- joint j21_elbow_pitch_r_joint: axis 0 1 0 -> 0.00272431 0.998023 -0.0627902; limit lower=-1.57 upper=1.57 effort=61 velocity=10.0 -> lower=-2.1948 upper=0.7374 effort=61 velocity=10.0; origin xyz=0 0 -0.2 rpy=0 0 0 -> xyz=0 -0.006598 -0.10487 rpy=0 0 0
- joint j22_elbow_yaw_r_joint: axis 0 0 1 -> -0.214789 0.0619088 0.974696; limit lower=-1.57 upper=1.57 effort=61 velocity=10.0 -> lower=-2.618 upper=2.618 effort=61 velocity=10.0; origin xyz=0 0 0 rpy=0 0 0 -> xyz=0.013817 -0.0097704 -0.1547 rpy=0 0 0
- joint j23_head_yaw_joint: limit lower=-1.57 upper=1.57 effort=61 velocity=10.0 -> lower=-0.6109 upper=0.6109 effort=61 velocity=10.0; origin xyz=0.1 0 0.2 rpy=0 0 0 -> xyz=-0.017638 0 0.2961 rpy=0 0 0
